Commit message: Adding Parte12

File: Parte11/psr_scara_p3_description/urdf/scara_p3.urdf (robot description, URDF)
Before this commit: robot scara_p3, 2 links, 1 joints
Links:
- link base_link: geometry visual cylinder length=1 radius=0.5
- link link1: geometry visual box size=4.0 1 1
Joints:
- removed joint base_link_to_lin1
- added joint base_link_to_link1: type continuous, parent base_link, child link1, origin xyz=0.0 0.0 2.0 rpy=0 0 0, axis 0 0 1
