Commit message: Adding Parte 14 and TH packages.

File: Parte12/p_moliveira_description_tp/urdf/p_moliveira.gazebo.xacro (robot description, xacro)
@@ -7,6 +7,7 @@
 <!--    <material>Gazebo/Yellow</material>-->
 <!--    <material>Gazebo/SarasColor</material>-->
-<!--    <material>Gazebo/Yellow</material>-->
-    <material>Gazebo/Bricks</material>
+    <material>Gazebo/Yellow</material>
+    <material>Gazebo/${player_color}</material>
+<!--    <material>Gazebo/Bricks</material>-->
   </gazebo>
   <gazebo reference="wheel_left_link">
@@ -144,7 +145,7 @@
       <visualize>$(arg camera_visual)</visualize>
       <camera>
-          <horizontal_fov>1.085595</horizontal_fov>
+          <horizontal_fov>2.085595</horizontal_fov>
           <image>
-              <width>640</width>
+              <width>1280</width>
               <height>480</height>
               <format>R8G8B8</format>

File: Parte12/p_moliveira_description_tp/urdf/p_moliveira.urdf.xacro (robot description, xacro)
@@ -1,28 +1,16 @@
 <?xml version="1.0" ?>
-<robot name="turtlebot3_waffle_pi" xmlns:xacro="http://ros.org/wiki/xacro">
-<!--  <xacro:include filename="$(find turtlebot3_description)/urdf/common_properties.xacro"/>-->
+<robot name="team_hunt_player" xmlns:xacro="http://ros.org/wiki/xacro">
+<!--  Arguments-->
+<!--  Arguments are used as: $(arg argument)-->
+  <xacro:arg name="player_name"  default="p_moliveira"/>
+  <xacro:arg name="player_color"  default="Red"/>
+<!-- Copy arguments to properties so that they are visible in the included xacros-->
+<!--  Properties are used as ${property}-->
+  <xacro:property name="player_name" value="$(arg player_name)"/>
+  <xacro:property name="player_color" value="$(arg player_color)"/>
+<!--  Includes-->
   <xacro:include filename="$(find p_moliveira_description_tp)/urdf/properties.xacro"/>
-<!--  <xacro:include filename="$(find turtlebot3_description)/urdf/turtlebot3_waffle_pi.gazebo.xacro"/>-->
   <xacro:include filename="$(find p_moliveira_description_tp)/urdf/p_moliveira.gazebo.xacro"/>
-<!--    <xacro:include filename="$(find p_moliveira_description)/urdf/player.gazebo.macro.xacro"/>-->
-<!--  <xacro:gazebo_macro player_color="$(arg player_color)" laser_visual="false" camera_visual="false" imu_visual="true"/>-->
-  <!-- Tables properties-->
-  <xacro:property name="M_PI" value="3.1415926535897931" />
-  <xacro:property name="table_height" value="0.795"/>
-  <xacro:property name="table_width" value=".9"/>
-  <xacro:property name="table_lenght" value="0.9"/>
-  <xacro:property name="table_tabletop_thickness" value="0.015"/>
-  <xacro:property name="table_leg_radius" value="0.02"/>
-  <xacro:include filename="$(find p_moliveira_description_tp)/urdf/table.macro.xacro"/>
-  <xacro:table_macro name="table" parent="base_link" width="${table_width}"
-                       lenght="${table_lenght}" height="${table_height}"
-                       tabletop_thickness="${table_tabletop_thickness}" leg_radius="${table_leg_radius}">
-        <origin xyz="-1 0 0" rpy="0 0 ${M_PI/2}" />
-  </xacro:table_macro>
-  <xacro:table_macro name="table2" parent="base_link" width="${table_width}"
-                       lenght="${table_lenght}" height="${table_height}"
-                       tabletop_thickness="${table_tabletop_thickness}" leg_radius="${table_leg_radius}">
-        <origin xyz="-1 0 3" rpy="0 0 ${M_PI/2}" />
-  </xacro:table_macro>
+<!--  Define links and joints-->
   <link name="base_footprint"/>
   <joint name="base_joint" type="fixed">
@@ -38,5 +26,5 @@
       </geometry>
 <!--      <material name="light_black"/>-->
-      <material name="sarascolor"/>
+      <material name="$(arg player_color)"/>
     </visual>
     <collision>
@@ -67,5 +55,6 @@
         <mesh filename="package://turtlebot3_description/meshes/wheels/left_tire.stl" scale="0.001 0.001 0.001"/>
       </geometry>
-      <material name="dark"/>
+<!--      <material name="dark"/>-->
+      <material name="Yellow"/>
     </visual>
     <collision>
@@ -95,5 +84,6 @@
         <mesh filename="package://turtlebot3_description/meshes/wheels/right_tire.stl" scale="0.001 0.001 0.001"/>
       </geometry>
-      <material name="dark"/>
+<!--      <material name="dark"/>-->
+      <material name="Yellow"/>
     </visual>
     <collision>
@@ -185,5 +175,6 @@
   </link>
   <joint name="camera_joint" type="fixed">
-    <origin xyz="0.073 -0.011 0.084" rpy="0 0 0"/>
+<!--    <origin xyz="0.073 -0.011 0.084" rpy="0 0 0"/>-->
+    <origin xyz="0.073 -0.011 0.584" rpy="0 0.45 0"/>
     <parent link="base_link"/>
     <child link="camera_link"/>

File: Parte12/p_moliveira_description_tp/urdf/properties.xacro (robot description, xacro)
@@ -12,3 +12,13 @@
         <color rgba="0.2 0.5 0.8 1.0"/>
     </material>
+    <!--    Team hunt player colors-->
+    <material name="Red">
+    <color rgba="1.0 0.0 0.0 1.0"/>
+    </material>
+    <material name="Green">
+    <color rgba="0.0 1.0 0.0 1.0"/>
+    </material>
+    <material name="Blue">
+    <color rgba="0.0 0.0 1.0 1.0"/>
+    </material>
 </robot>
